Commit message: added wildos light version planner

File: install/go2_sim/share/go2_sim/urdf/const.xacro (robot description, xacro)
@@ -1 +1,108 @@
-/anubi/src/go2_sim/urdf/const.xacro
+<?xml version="1.0"?>
+<!--
+  const.xacro
+  Robot dimension and inertia constants for the Unitree Go2.
+  Source: khaledgabr77/unitree_go2_ros2 / unitree_go2_description/urdf/const.xacro
+  Ported to: go2_sim (Gazebo Fortress, ROS 2 Humble)
+  No values were invented — all copied verbatim from source.
+-->
+<robot xmlns:xacro="http://www.ros.org/wiki/xacro">
+    <!-- ──── Numeric constant ──── -->
+    <xacro:property name="PI" value="3.1415926535897931"/>
+    <xacro:property name="stick_mass" value="0.00001"/>
+    <!-- ──── Simplified collision geometry ──── -->
+    <xacro:property name="trunk_width"  value="0.0935"/>
+    <xacro:property name="trunk_length" value="0.3762"/>
+    <xacro:property name="trunk_height" value="0.114"/>
+    <xacro:property name="hip_radius"   value="0.046"/>
+    <xacro:property name="hip_length"   value="0.04"/>
+    <xacro:property name="thigh_shoulder_radius" value="0.041"/>
+    <xacro:property name="thigh_shoulder_length" value="0.032"/>
+    <xacro:property name="thigh_width"  value="0.0245"/>
+    <xacro:property name="thigh_height" value="0.034"/>
+    <xacro:property name="calf_width"   value="0.016"/>
+    <xacro:property name="calf_height"  value="0.016"/>
+    <xacro:property name="foot_radius"  value="0.02"/>
+    <xacro:property name="stick_radius" value="0.01"/>
+    <xacro:property name="stick_length" value="0.2"/>
+    <!-- ──── Kinematic lengths ──── -->
+    <xacro:property name="thigh_offset" value="0.0955"/>
+    <xacro:property name="thigh_length" value="0.213"/>
+    <xacro:property name="calf_length"  value="0.213"/>
+    <!-- ──── Leg offsets from trunk centre ──── -->
+    <xacro:property name="leg_offset_x" value="0.1934"/>
+    <xacro:property name="leg_offset_y" value="0.0465"/>
+    <xacro:property name="hip_offset"   value="0.0955"/>
+    <!-- Explicit per-axis offsets (redundant with above, kept for readability) -->
+    <xacro:property name="hip_offset_x" value="0.1934"/>
+    <xacro:property name="hip_offset_y" value="0.0465"/>
+    <xacro:property name="hip_offset_z" value="0.0"/>
+    <xacro:property name="thigh_offset_x" value="0"/>
+    <xacro:property name="thigh_offset_y" value="0.0955"/>
+    <xacro:property name="thigh_offset_z" value="0.0"/>
+    <xacro:property name="calf_offset_x" value="0.0"/>
+    <xacro:property name="calf_offset_y" value="0.0"/>
+    <xacro:property name="calf_offset_z" value="-0.213"/>
+    <!-- ──── Joint limits ──── -->
+    <xacro:property name="damping"  value="0.01"/>
+    <xacro:property name="friction" value="0.2"/>
+    <xacro:property name="hip_position_max"   value="1.0472"/>
+    <xacro:property name="hip_position_min"   value="-1.0472"/>
+    <xacro:property name="hip_velocity_max"   value="30.1"/>
+    <xacro:property name="hip_torque_max"     value="23.7"/>
+    <xacro:property name="thigh_position_max" value="3.4907"/>
+    <xacro:property name="thigh_position_min" value="-1.5708"/>
+    <xacro:property name="thigh_velocity_max" value="30.1"/>
+    <xacro:property name="thigh_torque_max"   value="23.7"/>
+    <xacro:property name="calf_position_max"  value="-0.83776"/>
+    <xacro:property name="calf_position_min"  value="-2.7227"/>
+    <xacro:property name="calf_velocity_max"  value="20.06"/>
+    <xacro:property name="calf_torque_max"    value="35.55"/>
+    <!-- ──── Inertial values ──── -->
+    <!-- trunk -->
+    <xacro:property name="trunk_mass"  value="6.921"/>
+    <xacro:property name="trunk_com_x" value="0.021112"/>
+    <xacro:property name="trunk_com_y" value="0.00"/>
+    <xacro:property name="trunk_com_z" value="-0.005366"/>
+    <xacro:property name="trunk_ixx"   value="0.02448"/>
+    <xacro:property name="trunk_ixy"   value="0.00012166"/>
+    <xacro:property name="trunk_ixz"   value="0.0014849"/>
+    <xacro:property name="trunk_iyy"   value="0.098077"/>
+    <xacro:property name="trunk_iyz"   value="-3.12E-05"/>
+    <xacro:property name="trunk_izz"   value="0.107"/>
+    <!-- hip (left-front reference; mirroring applied in leg macro) -->
+    <xacro:property name="hip_mass"   value="0.678"/>
+    <xacro:property name="hip_com_x"  value="-0.0054"/>
+    <xacro:property name="hip_com_y"  value="0.00194"/>
+    <xacro:property name="hip_com_z"  value="-0.000105"/>
+    <xacro:property name="hip_ixx"    value="0.00048"/>
+    <xacro:property name="hip_ixy"    value="-3.01E-06"/>
+    <xacro:property name="hip_ixz"    value="1.11E-06"/>
+    <xacro:property name="hip_iyy"    value="0.000884"/>
+    <xacro:property name="hip_iyz"    value="-1.42E-06"/>
+    <xacro:property name="hip_izz"    value="0.000596"/>
+    <!-- thigh -->
+    <xacro:property name="thigh_mass"  value="1.152"/>
+    <xacro:property name="thigh_com_x" value="-0.00374"/>
+    <xacro:property name="thigh_com_y" value="-0.0223"/>
+    <xacro:property name="thigh_com_z" value="-0.0327"/>
+    <xacro:property name="thigh_ixx"   value="0.00584"/>
+    <xacro:property name="thigh_ixy"   value="8.72E-05"/>
+    <xacro:property name="thigh_ixz"   value="-0.000289"/>
+    <xacro:property name="thigh_iyy"   value="0.0058"/>
+    <xacro:property name="thigh_iyz"   value="0.000808"/>
+    <xacro:property name="thigh_izz"   value="0.00103"/>
+    <!-- calf -->
+    <xacro:property name="calf_mass"   value="0.154"/>
+    <xacro:property name="calf_com_x"  value="0.00548"/>
+    <xacro:property name="calf_com_y"  value="-0.000975"/>
+    <xacro:property name="calf_com_z"  value="-0.115"/>
+    <xacro:property name="calf_ixx"    value="0.00108"/>
+    <xacro:property name="calf_ixy"    value="3.4E-07"/>
+    <xacro:property name="calf_ixz"    value="1.72E-05"/>
+    <xacro:property name="calf_iyy"    value="0.0011"/>
+    <xacro:property name="calf_iyz"    value="8.28E-06"/>
+    <xacro:property name="calf_izz"    value="3.29E-05"/>
+    <!-- foot -->
+    <xacro:property name="foot_mass" value="0.06"/>
+</robot>

File: install/go2_sim/share/go2_sim/urdf/go2_sim.urdf.xacro (robot description, xacro)
@@ -1 +1,262 @@
-/anubi/src/go2_sim/urdf/go2_sim.urdf.xacro
+<?xml version="1.0"?>
+<!--
+  go2_sim.urdf.xacro
+  Unitree Go2 — Gazebo Fortress (Ignition Gazebo 6) + CHAMP simulation model.
+  Port contract:
+    - Source:  khaledgabr77/unitree_go2_ros2 (Gazebo Harmonic, ROS 2 Jazzy)
+    - Target:  go2_sim (Gazebo Fortress / Ignition Gazebo 6, ROS 2 Humble)
+  Frame tree:
+    base_link (robot body — matches go2_description and go2_bringup convention)
+      ├── trunk                  (body visual/collision/inertia; floating_base joint)
+      ├── imu_link               (IMU sensor frame)
+      ├── {lf,rf,lh,rh}_hip_link → {lf,rf,lh,rh}_upper_leg_link
+      │                         → {lf,rf,lh,rh}_lower_leg_link
+      │                         → LF_FOOT / RF_FOOT / LH_FOOT / RH_FOOT (CHAMP)
+      └── lidar_l1_link          (Unitree L1 LiDAR; provided by sensor_models macro)
+  CHAMP requires four foot links named exactly: LF_FOOT RF_FOOT LH_FOOT RH_FOOT
+  These are generated by the leg macro in leg.xacro.
+  Fortress plugins used (all Classic libgazebo_ros_* plugins removed):
+    - ign_ros2_control-system          (joint trajectory effort control)
+    - ignition-gazebo-imu-system       (IMU sensor)
+    - ignition-gazebo-contact-system   (foot contact sensors)
+    - ignition-gazebo-joint-state-publisher-system  (/joint_states)
+    - ignition-gazebo-sensors-system   (gpu_lidar — in world SDF, handles L1)
+  Topics published (bridged to ROS via ros_ign_bridge in launch file):
+    /joint_states       — sensor_msgs/JointState
+    /imu/data           — sensor_msgs/Imu
+    /lidar/points     — sensor_msgs/PointCloud2   (from L1 lidar_l1 sensor)
+    /cmd_vel            — geometry_msgs/Twist        (ROS → Gazebo)
+  DO NOT USE libgazebo_ros_* plugins here — they are Gazebo Classic only.
+  DO NOT USE gz:: namespaces — Fortress uses ignition:: exclusively.
+-->
+<robot name="go2"
+       xmlns:xacro="http://www.ros.org/wiki/xacro">
+  <!-- ── xacro arguments ── -->
+  <xacro:arg name="DEBUG"            default="false"/>
+  <xacro:arg name="robot_controllers"
+             default="$(find go2_sim)/config/ros_control.yaml"/>
+  <!-- ── Include sub-files ── -->
+  <xacro:include filename="$(find go2_sim)/urdf/const.xacro"/>
+  <xacro:include filename="$(find go2_sim)/urdf/materials.xacro"/>
+  <xacro:include filename="$(find go2_sim)/urdf/leg.xacro"/>
+  <xacro:include filename="$(find sensor_models)/urdf/l1_lidar.urdf.xacro"/>
+  <!-- ════════════════════════════════════════════════════════════════════
+       GAZEBO PLUGINS  (Fortress / ignition:: namespace)
+       ════════════════════════════════════════════════════════════════════ -->
+  <!-- ign_ros2_control: loads controller_manager, reads ros_control.yaml -->
+  <gazebo>
+    <plugin filename="ign_ros2_control-system"
+            name="ign_ros2_control::IgnitionROS2ControlPlugin">
+      <parameters>$(arg robot_controllers)</parameters>
+      <robot_param_node>robot_state_publisher</robot_param_node>
+    </plugin>
+  </gazebo>
+  <!-- Joint state publisher: publishes /joint_states from sim -->
+  <gazebo>
+    <plugin filename="ignition-gazebo-joint-state-publisher-system"
+            name="ignition::gazebo::systems::JointStatePublisher">
+    </plugin>
+  </gazebo>
+  <!-- Ground-truth odometry (Fortress OdometryPublisher).
+       Publishes ignition.msgs.Odometry on Gazebo topic /odom, which the
+       ros_ign_bridge in sim_champ.launch.py remaps to ROS /odom/raw.
+       This gives the A* and MPC nodes a reliable ground-truth pose without
+       depending on CHAMP's leg-kinematic state estimator. -->
+  <gazebo>
+    <plugin filename="ignition-gazebo-odometry-publisher-system"
+            name="ignition::gazebo::systems::OdometryPublisher">
+      <odom_frame>odom</odom_frame>
+      <robot_base_frame>base_link</robot_base_frame>
+      <odom_topic>odom</odom_topic>
+      <dimensions>2</dimensions>
+    </plugin>
+  </gazebo>
+  <!-- ════════════════════════════════════════════════════════════════════
+       OPTIONAL DEBUG MODE: pin robot to world for tuning
+       ════════════════════════════════════════════════════════════════════ -->
+  <xacro:if value="$(arg DEBUG)">
+    <link name="world"/>
+    <joint name="base_static_joint" type="fixed">
+      <origin rpy="0 0 0" xyz="0 0 0"/>
+      <parent link="world"/>
+      <child link="base_link"/>
+    </joint>
+  </xacro:if>
+  <!-- ════════════════════════════════════════════════════════════════════
+       BASE LINK  (virtual root — matches CHAMP expectation)
+       ════════════════════════════════════════════════════════════════════ -->
+  <link name="base_link">
+    <visual>
+      <origin rpy="0 0 0" xyz="0 0 0"/>
+      <geometry><box size="0.001 0.001 0.001"/></geometry>
+    </visual>
+  </link>
+  <!-- ════════════════════════════════════════════════════════════════════
+       TRUNK  (main body visual / collision / inertia)
+       Mesh: base.dae  (byte-identical to source trunk.dae; same 10727399 B)
+       ════════════════════════════════════════════════════════════════════ -->
+  <joint name="floating_base" type="fixed">
+    <origin rpy="0 0 0" xyz="0 0 0"/>
+    <parent link="base_link"/>
+    <child link="trunk"/>
+  </joint>
+  <link name="trunk">
+    <visual>
+      <origin rpy="0 0 0" xyz="0 0 0"/>
+      <geometry>
+        <mesh filename="package://go2_sim/meshes/dae/base.dae" scale="1 1 1"/>
+      </geometry>
+    </visual>
+    <collision>
+      <origin rpy="0 0 0" xyz="0 0 0"/>
+      <geometry>
+        <box size="${trunk_length} ${trunk_width} ${trunk_height}"/>
+      </geometry>
+    </collision>
+    <inertial>
+      <origin rpy="0 0 0" xyz="${trunk_com_x} ${trunk_com_y} ${trunk_com_z}"/>
+      <mass value="${trunk_mass}"/>
+      <inertia ixx="${trunk_ixx}" ixy="${trunk_ixy}" ixz="${trunk_ixz}"
+               iyy="${trunk_iyy}" iyz="${trunk_iyz}" izz="${trunk_izz}"/>
+    </inertial>
+  </link>
+  <gazebo reference="trunk">
+    <mu1>0.2</mu1>
+    <mu2>0.2</mu2>
+    <kp>10000.0</kp>
+    <kd>1.0</kd>
+  </gazebo>
+  <!-- ════════════════════════════════════════════════════════════════════
+       IMU LINK
+       ════════════════════════════════════════════════════════════════════ -->
+  <joint name="imu_joint" type="fixed">
+    <parent link="trunk"/>
+    <child link="imu_link"/>
+    <origin rpy="0 0 0" xyz="0 0 0"/>
+  </joint>
+  <link name="imu_link">
+    <inertial>
+      <mass value="0.001"/>
+      <origin rpy="0 0 0" xyz="0 0 0"/>
+      <inertia ixx="0.0001" ixy="0" ixz="0" iyy="0.0001" iyz="0" izz="0.0001"/>
+    </inertial>
+    <visual>
+      <origin rpy="0 0 0" xyz="0 0 0"/>
+      <geometry><box size="0.001 0.001 0.001"/></geometry>
+    </visual>
+    <collision>
+      <origin rpy="0 0 0" xyz="0 0 0"/>
+      <geometry><box size="0.001 0.001 0.001"/></geometry>
+    </collision>
+  </link>
+  <!--
+    IMU sensor (Fortress syntax).
+    Published on topic: /imu/data
+    Bridged to ROS via ros_ign_bridge in sim_champ.launch.py.
+    System plugin ignition-gazebo-imu-system is loaded in the world SDF.
+  -->
+  <gazebo reference="imu_link">
+    <sensor name="imu_sensor" type="imu">
+      <always_on>1</always_on>
+      <update_rate>200</update_rate>
+      <topic>/imu/data</topic>
+      <ignition_frame_id>imu_link</ignition_frame_id>
+      <imu>
+        <angular_velocity>
+          <x><noise type="gaussian"><mean>0</mean><stddev>0.009</stddev></noise></x>
+          <y><noise type="gaussian"><mean>0</mean><stddev>0.009</stddev></noise></y>
+          <z><noise type="gaussian"><mean>0</mean><stddev>0.009</stddev></noise></z>
+        </angular_velocity>
+        <linear_acceleration>
+          <x><noise type="gaussian"><mean>0</mean><stddev>0.021</stddev></noise></x>
+          <y><noise type="gaussian"><mean>0</mean><stddev>0.021</stddev></noise></y>
+          <z><noise type="gaussian"><mean>0</mean><stddev>0.021</stddev></noise></z>
+        </linear_acceleration>
+      </imu>
+    </sensor>
+  </gazebo>
+  <!-- ════════════════════════════════════════════════════════════════════
+       LEGS  (4× instantiation via leg macro — defines foot links LF/RF/LH/RH_FOOT)
+       ════════════════════════════════════════════════════════════════════ -->
+  <!--  RF: mirror=-1 (right), mirror_dae=False (right mesh), front_hind=1, front_hind_dae=True  -->
+  <xacro:leg name="rf" mirror="-1" mirror_dae="False" front_hind="1"  front_hind_dae="True"/>
+  <!--  LF: mirror=1  (left),  mirror_dae=True  (left mesh),  front_hind=1, front_hind_dae=True  -->
+  <xacro:leg name="lf" mirror="1"  mirror_dae="True"  front_hind="1"  front_hind_dae="True"/>
+  <!--  RH: mirror=-1 (right), mirror_dae=False (right mesh), front_hind=-1, front_hind_dae=False -->
+  <xacro:leg name="rh" mirror="-1" mirror_dae="False" front_hind="-1" front_hind_dae="False"/>
+  <!--  LH: mirror=1  (left),  mirror_dae=True  (left mesh),  front_hind=-1, front_hind_dae=False -->
+  <xacro:leg name="lh" mirror="1"  mirror_dae="True"  front_hind="-1" front_hind_dae="False"/>
+  <!-- ── Gazebo physics properties for legs ── -->
+  <!-- LF leg -->
+  <gazebo reference="lf_hip_link">       <mu1>0.2</mu1><mu2>0.2</mu2></gazebo>
+  <gazebo reference="lf_upper_leg_link"> <mu1>0.2</mu1><mu2>0.2</mu2><self_collide>1</self_collide><kp>10000.0</kp><kd>1.0</kd></gazebo>
+  <gazebo reference="lf_lower_leg_link"> <mu1>0.2</mu1><mu2>0.2</mu2><self_collide>1</self_collide></gazebo>
+  <gazebo reference="LF_FOOT">           <mu1>0.6</mu1><mu2>0.6</mu2><self_collide>1</self_collide><kp>10000.0</kp><kd>1.0</kd></gazebo>
+  <!-- RF leg -->
+  <gazebo reference="rf_hip_link">       <mu1>0.2</mu1><mu2>0.2</mu2></gazebo>
+  <gazebo reference="rf_upper_leg_link"> <mu1>0.2</mu1><mu2>0.2</mu2><self_collide>1</self_collide><kp>10000.0</kp><kd>1.0</kd></gazebo>
+  <gazebo reference="rf_lower_leg_link"> <mu1>0.2</mu1><mu2>0.2</mu2><self_collide>1</self_collide></gazebo>
+  <gazebo reference="RF_FOOT">           <mu1>0.6</mu1><mu2>0.6</mu2><self_collide>1</self_collide><kp>10000.0</kp><kd>1.0</kd></gazebo>
+  <!-- LH leg -->
+  <gazebo reference="lh_hip_link">       <mu1>0.2</mu1><mu2>0.2</mu2></gazebo>
+  <gazebo reference="lh_upper_leg_link"> <mu1>0.2</mu1><mu2>0.2</mu2><self_collide>1</self_collide><kp>10000.0</kp><kd>1.0</kd></gazebo>
+  <gazebo reference="lh_lower_leg_link"> <mu1>0.2</mu1><mu2>0.2</mu2><self_collide>1</self_collide></gazebo>
+  <gazebo reference="LH_FOOT">           <mu1>0.6</mu1><mu2>0.6</mu2><self_collide>1</self_collide><kp>10000.0</kp><kd>1.0</kd></gazebo>
+  <!-- RH leg -->
+  <gazebo reference="rh_hip_link">       <mu1>0.2</mu1><mu2>0.2</mu2></gazebo>
+  <gazebo reference="rh_upper_leg_link"> <mu1>0.2</mu1><mu2>0.2</mu2><self_collide>1</self_collide><kp>10000.0</kp><kd>1.0</kd></gazebo>
+  <gazebo reference="rh_lower_leg_link"> <mu1>0.2</mu1><mu2>0.2</mu2><self_collide>1</self_collide></gazebo>
+  <gazebo reference="RH_FOOT">           <mu1>0.6</mu1><mu2>0.6</mu2><self_collide>1</self_collide><kp>10000.0</kp><kd>1.0</kd></gazebo>
+  <!-- ════════════════════════════════════════════════════════════════════
+       FOOT CONTACT SENSORS  (Fortress syntax, ignition-gazebo-contact-system)
+       One sensor per foot; collision name = <foot_link>_collision (auto-generated
+       by Gazebo from the URDF collision element of each foot link).
+       ════════════════════════════════════════════════════════════════════ -->
+  <gazebo reference="LF_FOOT">
+    <sensor name="LF_FOOT_contact" type="contact">
+      <always_on>1</always_on>
+      <contact>
+        <collision>LF_FOOT_collision</collision>
+      </contact>
+    </sensor>
+  </gazebo>
+  <gazebo reference="RF_FOOT">
+    <sensor name="RF_FOOT_contact" type="contact">
+      <always_on>1</always_on>
+      <contact>
+        <collision>RF_FOOT_collision</collision>
+      </contact>
+    </sensor>
+  </gazebo>
+  <gazebo reference="LH_FOOT">
+    <sensor name="LH_FOOT_contact" type="contact">
+      <always_on>1</always_on>
+      <contact>
+        <collision>LH_FOOT_collision</collision>
+      </contact>
+    </sensor>
+  </gazebo>
+  <gazebo reference="RH_FOOT">
+    <sensor name="RH_FOOT_contact" type="contact">
+      <always_on>1</always_on>
+      <contact>
+        <collision>RH_FOOT_collision</collision>
+      </contact>
+    </sensor>
+  </gazebo>
+  <!-- ════════════════════════════════════════════════════════════════════
+       L1 LIDAR  (from sensor_models Fortress macro)
+       Mount position from source repo reference
+       (unitree_ros/go2_description.urdf radar_joint):
+         xyz = (0.28945, 0, -0.046825) relative to base_link
+       The macro creates lidar_link (with prefix="") and publishes on
+       Ignition topic /unilidar/cloud/points, bridged to ROS /lidar/points.
+       Frame "lidar_link" matches:
+         scan_from_cloud.yaml  target_frame: lidar_link
+         go2_description       lidar_link frame convention
+         nav2_params.yaml      voxel_layer expects /lidar/points in lidar_link
+       ════════════════════════════════════════════════════════════════════ -->
+  <xacro:l1_lidar parent="base_link" prefix="">
+    <origin xyz="0.28945 0 -0.046825" rpy="0 0 0"/>
+  </xacro:l1_lidar>
+</robot>
