Commit message: added wildos light version planner

File: install/go2_sim/share/go2_sim/urdf/leg.xacro (robot description, xacro)
@@ -1 +1,241 @@
-/anubi/src/go2_sim/urdf/leg.xacro
+<?xml version="1.0"?>
+<!--
+  leg.xacro
+  Parametric leg macro for the Unitree Go2 (Gazebo Fortress / ign_ros2_control).
+  Source: khaledgabr77/unitree_go2_ros2 / unitree_go2_description/urdf/leg.xacro
+  Changes vs. source:
+    1. Foot link names renamed: {name}_foot_link → uppercase CHAMP convention
+         lf → LF_FOOT,  rf → RF_FOOT,  lh → LH_FOOT,  rh → RH_FOOT
+       Joint child references updated accordingly.
+    2. ros2_control hardware plugin changed:
+         Fortress control interface plugin → ign_ros2_control/IgnitionSystem
+    3. Mesh paths changed:
+         package://unitree_go2_description/meshes/ → package://go2_sim/meshes/dae/
+    4. Typo in source fixed: line had `type="fixed">0` — the stray `0` removed.
+  Macro parameters (unchanged from source):
+    name         — leg prefix: lf | rf | lh | rh
+    mirror       — Y-axis sign:  1 (left) | -1 (right)
+    mirror_dae   — True (left, use original mesh) | False (right, use mirrored mesh)
+    front_hind   — X-axis sign:  1 (front) | -1 (hind)
+    front_hind_dae — True (front) | False (hind)
+-->
+<robot xmlns:xacro="http://www.ros.org/wiki/xacro">
+    <!--
+      Foot link name map (CHAMP convention, uppercase):
+        lf_foot_link → LF_FOOT
+        rf_foot_link → RF_FOOT
+        lh_foot_link → LH_FOOT
+        rh_foot_link → RH_FOOT
+      The xacro property below derives the CHAMP name from the leg prefix.
+    -->
+    <xacro:macro name="leg" params="name mirror mirror_dae front_hind front_hind_dae">
+        <!-- Derive CHAMP-convention foot link name from leg prefix -->
+        <xacro:if value="${name == 'lf'}">
+            <xacro:property name="foot_link_name" value="LF_FOOT"/>
+        </xacro:if>
+        <xacro:if value="${name == 'rf'}">
+            <xacro:property name="foot_link_name" value="RF_FOOT"/>
+        </xacro:if>
+        <xacro:if value="${name == 'lh'}">
+            <xacro:property name="foot_link_name" value="LH_FOOT"/>
+        </xacro:if>
+        <xacro:if value="${name == 'rh'}">
+            <xacro:property name="foot_link_name" value="RH_FOOT"/>
+        </xacro:if>
+        <!-- ── Hip joint ── -->
+        <joint name="${name}_hip_joint" type="revolute">
+            <xacro:if value="${(mirror_dae == False) and (front_hind_dae == True)}">
+                <origin rpy="0 0 0" xyz="${leg_offset_x} ${-leg_offset_y} 0"/>
+            </xacro:if>
+            <xacro:if value="${(mirror_dae == True) and (front_hind_dae == True)}">
+                <origin rpy="0 0 0" xyz="${leg_offset_x} ${leg_offset_y} 0"/>
+            </xacro:if>
+            <xacro:if value="${(mirror_dae == False) and (front_hind_dae == False)}">
+                <origin rpy="0 0 0" xyz="${-leg_offset_x} ${-leg_offset_y} 0"/>
+            </xacro:if>
+            <xacro:if value="${(mirror_dae == True) and (front_hind_dae == False)}">
+                <origin rpy="0 0 0" xyz="${-leg_offset_x} ${leg_offset_y} 0"/>
+            </xacro:if>
+            <parent link="trunk"/>
+            <child link="${name}_hip_link"/>
+            <axis xyz="1 0 0"/>
+            <dynamics damping="${damping}" friction="${friction}"/>
+            <xacro:if value="${(mirror_dae == True)}">
+                <limit effort="${hip_torque_max}" velocity="${hip_velocity_max}"
+                       lower="${hip_position_min}" upper="${hip_position_max}"/>
+            </xacro:if>
+            <xacro:if value="${(mirror_dae == False)}">
+                <limit effort="${hip_torque_max}" velocity="${hip_velocity_max}"
+                       lower="${-hip_position_max}" upper="${-hip_position_min}"/>
+            </xacro:if>
+        </joint>
+        <!-- ── Hip link ── -->
+        <link name="${name}_hip_link">
+            <visual>
+                <xacro:if value="${(mirror_dae == True) and (front_hind_dae == True)}">
+                    <origin rpy="0 0 0" xyz="0 0 0"/>
+                </xacro:if>
+                <xacro:if value="${(mirror_dae == False) and (front_hind_dae == True)}">
+                    <origin rpy="${PI} 0 0" xyz="0 0 0"/>
+                </xacro:if>
+                <xacro:if value="${(mirror_dae == True) and (front_hind_dae == False)}">
+                    <origin rpy="0 ${PI} 0" xyz="0 0 0"/>
+                </xacro:if>
+                <xacro:if value="${(mirror_dae == False) and (front_hind_dae == False)}">
+                    <origin rpy="${PI} ${PI} 0" xyz="0 0 0"/>
+                </xacro:if>
+                <geometry>
+                    <mesh filename="package://go2_sim/meshes/dae/hip.dae" scale="1 1 1"/>
+                </geometry>
+            </visual>
+            <collision>
+                <origin rpy="${PI/2.0} 0 0" xyz="0 ${hip_offset*mirror} 0"/>
+                <geometry>
+                    <cylinder length="${hip_length}" radius="${hip_radius}"/>
+                </geometry>
+            </collision>
+            <inertial>
+                <origin rpy="0 0 0"
+                        xyz="${hip_com_x*front_hind} ${hip_com_y*mirror} ${hip_com_z}"/>
+                <mass value="${hip_mass}"/>
+                <inertia
+                    ixx="${hip_ixx}"
+                    ixy="${hip_ixy*mirror*front_hind}"
+                    ixz="${hip_ixz*front_hind}"
+                    iyy="${hip_iyy}"
+                    iyz="${hip_iyz*mirror}"
+                    izz="${hip_izz}"/>
+            </inertial>
+        </link>
+        <!-- ── Upper leg joint ── -->
+        <joint name="${name}_upper_leg_joint" type="revolute">
+            <origin rpy="0 0 0" xyz="0 ${thigh_offset*mirror} 0"/>
+            <parent link="${name}_hip_link"/>
+            <child link="${name}_upper_leg_link"/>
+            <axis xyz="0 1 0"/>
+            <dynamics damping="${damping}" friction="${friction}"/>
+            <limit effort="${thigh_torque_max}" velocity="${thigh_velocity_max}"
+                   lower="${thigh_position_min}" upper="${thigh_position_max}"/>
+        </joint>
+        <!-- ── Upper leg link ── -->
+        <link name="${name}_upper_leg_link">
+            <visual>
+                <origin rpy="0 0 0" xyz="0 0 0"/>
+                <geometry>
+                    <xacro:if value="${mirror_dae == True}">
+                        <mesh filename="package://go2_sim/meshes/dae/thigh.dae" scale="1 1 1"/>
+                    </xacro:if>
+                    <xacro:if value="${mirror_dae == False}">
+                        <mesh filename="package://go2_sim/meshes/dae/thigh_mirror.dae" scale="1 1 1"/>
+                    </xacro:if>
+                </geometry>
+            </visual>
+            <collision>
+                <origin rpy="0 ${PI/2.0} 0" xyz="0 0 ${-thigh_length/2.0}"/>
+                <geometry>
+                    <box size="${thigh_length} ${thigh_width} ${thigh_height}"/>
+                </geometry>
+            </collision>
+            <inertial>
+                <origin rpy="0 0 0"
+                        xyz="${thigh_com_x} ${thigh_com_y*mirror} ${thigh_com_z}"/>
+                <mass value="${thigh_mass}"/>
+                <inertia
+                    ixx="${thigh_ixx}"
+                    ixy="${thigh_ixy*mirror}"
+                    ixz="${thigh_ixz}"
+                    iyy="${thigh_iyy}"
+                    iyz="${thigh_iyz*mirror}"
+                    izz="${thigh_izz}"/>
+            </inertial>
+        </link>
+        <!-- ── Lower leg joint ── -->
+        <joint name="${name}_lower_leg_joint" type="revolute">
+            <origin rpy="0 0 0" xyz="0 0 ${-thigh_length}"/>
+            <parent link="${name}_upper_leg_link"/>
+            <child link="${name}_lower_leg_link"/>
+            <axis xyz="0 1 0"/>
+            <dynamics damping="${damping}" friction="${friction}"/>
+            <limit effort="${calf_torque_max}" velocity="${calf_velocity_max}"
+                   lower="${calf_position_min}" upper="${calf_position_max}"/>
+        </joint>
+        <!-- ── Lower leg link ── -->
+        <link name="${name}_lower_leg_link">
+            <visual>
+                <origin rpy="0 0 0" xyz="0 0 0"/>
+                <geometry>
+                    <mesh filename="package://go2_sim/meshes/dae/calf.dae" scale="1 1 1"/>
+                </geometry>
+            </visual>
+            <collision>
+                <origin rpy="0 ${PI/2.0} 0" xyz="0 0 ${-calf_length/2.0}"/>
+                <geometry>
+                    <box size="${calf_length} ${calf_width} ${calf_height}"/>
+                </geometry>
+            </collision>
+            <inertial>
+                <origin rpy="0 0 0"
+                        xyz="${calf_com_x} ${calf_com_y} ${calf_com_z}"/>
+                <mass value="${calf_mass}"/>
+                <inertia
+                    ixx="${calf_ixx}"
+                    ixy="${calf_ixy}"
+                    ixz="${calf_ixz}"
+                    iyy="${calf_iyy}"
+                    iyz="${calf_iyz}"
+                    izz="${calf_izz}"/>
+            </inertial>
+        </link>
+        <!-- ── Foot joint  (child = CHAMP uppercase foot link name) ── -->
+        <joint name="${name}_foot_joint" type="fixed">
+            <origin rpy="0 0 0" xyz="0 0 ${-(calf_length)}"/>
+            <parent link="${name}_lower_leg_link"/>
+            <child link="${foot_link_name}"/>
+        </joint>
+        <!-- ── Foot link  (CHAMP-convention uppercase name) ── -->
+        <link name="${foot_link_name}">
+            <visual>
+                <origin rpy="0 0 0" xyz="0 0 0"/>
+                <geometry>
+                    <sphere radius="${foot_radius-0.01}"/>
+                </geometry>
+            </visual>
+            <collision>
+                <origin rpy="0 0 0" xyz="0 0 0"/>
+                <geometry>
+                    <sphere radius="${foot_radius}"/>
+                </geometry>
+            </collision>
+            <inertial>
+                <mass value="${foot_mass}"/>
+                <inertia
+                    ixx="${(2*foot_mass)/5.0*(foot_radius*foot_radius)}"
+                    ixy="0.0" ixz="0.0"
+                    iyy="${(2*foot_mass)/5.0*(foot_radius*foot_radius)}"
+                    iyz="0.0"
+                    izz="${(2*foot_mass)/5.0*(foot_radius*foot_radius)}"/>
+            </inertial>
+        </link>
+        <!-- ── ros2_control interface (Fortress: ign_ros2_control/IgnitionSystem) ── -->
+        <ros2_control name="${name}" type="system">
+            <hardware>
+                <plugin>ign_ros2_control/IgnitionSystem</plugin>
+            </hardware>
+            <joint name="${name}_hip_joint">
+                <command_interface name="effort"/>
+                <state_interface name="position"/>
+                <state_interface name="velocity"/>
+            </joint>
+            <joint name="${name}_upper_leg_joint">
+                <command_interface name="effort"/>
+                <state_interface name="position"/>
+                <state_interface name="velocity"/>
+            </joint>
+            <joint name="${name}_lower_leg_joint">
+                <command_interface name="effort"/>
+                <state_interface name="position"/>
+                <state_interface name="velocity"/>
+            </joint>
+        </ros2_control>
+    </xacro:macro>
+</robot>

File: install/go2_sim/share/go2_sim/urdf/materials.xacro (robot description, xacro)
@@ -1 +1,36 @@
-/anubi/src/go2_sim/urdf/materials.xacro
+<?xml version="1.0"?>
+<!--
+  materials.xacro
+  URDF material definitions for the Unitree Go2.
+  Source: khaledgabr77/unitree_go2_ros2 / unitree_go2_description/urdf/materials.xacro
+  Ported verbatim — no changes.
+-->
+<robot>
+    <material name="black">
+        <color rgba="0.0 0.0 0.0 1.0"/>
+    </material>
+    <material name="blue">
+        <color rgba="0.0 0.0 0.8 1.0"/>
+    </material>
+    <material name="green">
+        <color rgba="0.0 0.8 0.0 1.0"/>
+    </material>
+    <material name="grey">
+        <color rgba="0.2 0.2 0.2 0.0"/>
+    </material>
+    <material name="silver">
+        <color rgba="${233/255} ${233/255} ${216/255} 1.0"/>
+    </material>
+    <material name="orange">
+        <color rgba="${255/255} ${108/255} ${10/255} 1.0"/>
+    </material>
+    <material name="brown">
+        <color rgba="${222/255} ${207/255} ${195/255} 1.0"/>
+    </material>
+    <material name="red">
+        <color rgba="0.8 0.0 0.0 1.0"/>
+    </material>
+    <material name="white">
+        <color rgba="1.0 1.0 1.0 1.0"/>
+    </material>
+</robot>
