Commit message: new version of wildos planner

File: src/go2_description/urdf/go2.urdf.xacro (robot description, xacro)
@@ -170,4 +170,60 @@
   </link>
   <!-- ═══════════════════════════════════════════════════════════════════════
+       STEREO CAMERA FRAMES  —  TF frames for real-robot deployment.
+       No Gazebo sensors here; the physical camera driver publishes its own
+       topics.  These frames must match the mount position used in go2_sim so
+       that cloud_self_filter.py stereo_to_lidar_d{x,y,z} offsets are the same
+       in simulation and on hardware.
+       Mount: xyz=(0.265, 0.0, 0.12) from base_link, baseline=0.12 m
+         stereo_camera_link — bar midpoint (parent of left/right)
+         stereo_left_link   — left optic centre  (+Y offset = baseline/2 = 0.06 m)
+         stereo_right_link  — right optic centre (-Y offset)
+  ════════════════════════════════════════════════════════════════════════════ -->
+  <joint name="base_link_to_stereo_camera" type="fixed">
+    <parent link="base_link"/>
+    <child  link="stereo_camera_link"/>
+    <origin xyz="0.265 0.0 0.12" rpy="0 0 0"/>
+  </joint>
+  <link name="stereo_camera_link">
+    <visual>
+      <geometry><box size="0.030 0.140 0.030"/></geometry>
+      <material name="dark_grey"/>
+    </visual>
+    <inertial>
+      <mass value="0.10"/>
+      <inertia ixx="0.0001" ixy="0" ixz="0" iyy="0.0001" iyz="0" izz="0.0001"/>
+    </inertial>
+  </link>
+  <joint name="stereo_camera_to_left" type="fixed">
+    <parent link="stereo_camera_link"/>
+    <child  link="stereo_left_link"/>
+    <origin xyz="0 0.06 0" rpy="0 0 0"/>
+  </joint>
+  <link name="stereo_left_link">
+    <visual>
+      <geometry><box size="0.020 0.020 0.020"/></geometry>
+      <material name="dark_grey"/>
+    </visual>
+    <inertial>
+      <mass value="0.010"/>
+      <inertia ixx="1e-5" ixy="0" ixz="0" iyy="1e-5" iyz="0" izz="1e-5"/>
+    </inertial>
+  </link>
+  <joint name="stereo_camera_to_right" type="fixed">
+    <parent link="stereo_camera_link"/>
+    <child  link="stereo_right_link"/>
+    <origin xyz="0 -0.06 0" rpy="0 0 0"/>
+  </joint>
+  <link name="stereo_right_link">
+    <visual>
+      <geometry><box size="0.020 0.020 0.020"/></geometry>
+      <material name="dark_grey"/>
+    </visual>
+    <inertial>
+      <mass value="0.010"/>
+      <inertia ixx="1e-5" ixy="0" ixz="0" iyy="1e-5" iyz="0" izz="1e-5"/>
+    </inertial>
+  </link>
+  <!-- ═══════════════════════════════════════════════════════════════════════
        Gazebo plugins  (only included when use_gazebo:=true)
        TODO(sim): Replace stubs with working Gazebo Humble plugins.

File: src/go2_sim/urdf/go2_sim.urdf.xacro (robot description, xacro)
@@ -41,4 +41,5 @@
   <xacro:include filename="$(find go2_sim)/urdf/leg.xacro"/>
   <xacro:include filename="$(find sensor_models)/urdf/l1_lidar.urdf.xacro"/>
+  <xacro:include filename="$(find sensor_models)/urdf/stereo_camera.urdf.xacro"/>
   <!-- ════════════════════════════════════════════════════════════════════
        GAZEBO PLUGINS  (Fortress / ignition:: namespace)
@@ -260,3 +261,23 @@
     <origin xyz="0.28945 0 -0.046825" rpy="0 0 0"/>
   </xacro:l1_lidar>
+  <!-- ════════════════════════════════════════════════════════════════════
+       STEREO CAMERA  (from sensor_models Fortress macro)
+       Mounted on the front face of the body, above the LiDAR.
+         xyz = (0.265, 0.0, 0.12) relative to base_link
+         baseline = 0.12 m  →  left at y=+0.06, right at y=-0.06
+       Ignition topics (bridged to ROS in sim_champ.launch.py):
+         /stereo/left/image_raw      — left RGB image
+         /stereo/left/camera_info    — left camera info
+         /stereo/depth_image         — depth image (float32 m)
+         /stereo/points              — PointCloud2 → merged into /lidar/points_filtered
+         /stereo/right/image_raw     — right RGB image
+         /stereo/right/camera_info   — right camera info
+       cloud_self_filter (stereo_to_lidar_d{x,y,z}):
+         dx = lidar_x - cam_x  = 0.28945 - 0.265       = +0.02445 m
+         dy = lidar_y - left_y = 0.0     - 0.06        = -0.06000 m
+         dz = lidar_z - cam_z  = -0.046825 - 0.12      = -0.16683 m
+       ════════════════════════════════════════════════════════════════════ -->
+  <xacro:stereo_camera parent="base_link" prefix="stereo" baseline="0.12">
+    <origin xyz="0.265 0.0 0.12" rpy="0 0 0"/>
+  </xacro:stereo_camera>
 </robot>
